File: panel/1u-mult-panel.kicad_pcb (KiCad board)
At the start: 2 copper layers, 30 x 39.6 mm, 10 parts

Commit message: Enlarge holes, add mounting holes, add silkscreen in/out markings
Parts:
- added ?: , Wire_Pads:SolderWirePad_single_0-8mmDrill, F.Cu at (7.50, 17.0)
- added ?: , Wire_Pads:SolderWirePad_single_0-8mmDrill, F.Cu at (-7.50, -6.52)
- moved ? 18.2 mm to (7.50, -16.8)
